File: discrete_filter_board/generic_filt_v1/generic_filt_v1.kicad_pcb (KiCad board)
At the start: 2 copper layers, 35.4 x 14.9 mm, 53 parts, among them J1 Conn_Coaxial, J2 Conn_Coaxial, J3 Conn_Coaxial, J4 Conn_Coaxial, J5 Conn_Coaxial, J6 Conn_Coaxial, J7 Conn_Coaxial, J8 Conn_Coaxial, U1 PGA-103+

Commit message: completed pcb routing
Parts:
- added H10: MountingHole_Pad, MountingHole:MountingHole_2.2mm_M2_Pad_Via, F.Cu at (152.3, 73.4)
- added H11: MountingHole_Pad, MountingHole:MountingHole_2.2mm_M2_Pad_Via, F.Cu at (141.6, 83.6)
- added H12: MountingHole_Pad, MountingHole:MountingHole_2.2mm_M2_Pad_Via, F.Cu at (152.3, 83.6)
- added H13: MountingHole_Pad, MountingHole:MountingHole_2.2mm_M2_Pad_Via, F.Cu at (137.4, 112.6)
- added H14: MountingHole_Pad, MountingHole:MountingHole_2.2mm_M2_Pad_Via, F.Cu at (148.6, 92.6)
- added H15: MountingHole_Pad, MountingHole:MountingHole_2.2mm_M2_Pad_Via, F.Cu at (137.5, 92.6)
- added H16: MountingHole_Pad, MountingHole:MountingHole_2.2mm_M2_Pad_Via, F.Cu at (148.6, 112.6)
- added H17: MountingHole_Pad, MountingHole:MountingHole_2.2mm_M2_Pad_Via, F.Cu at (159.3, 92.6)
- added H18: MountingHole_Pad, MountingHole:MountingHole_2.2mm_M2_Pad_Via, F.Cu at (159.3, 112.6)
- added H19: MountingHole_Pad, MountingHole:MountingHole_2.2mm_M2_Pad_Via, F.Cu at (135.5, 122.1)
- added H20: MountingHole_Pad, MountingHole:MountingHole_2.2mm_M2_Pad_Via, F.Cu at (144.5, 122.1)
- added H21: MountingHole_Pad, MountingHole:MountingHole_2.2mm_M2_Pad_Via, F.Cu at (135.7, 142.1)
- added H22: MountingHole_Pad, MountingHole:MountingHole_2.2mm_M2_Pad_Via, F.Cu at (159.4, 142.1)
- added H23: MountingHole_Pad, MountingHole:MountingHole_2.2mm_M2_Pad_Via, F.Cu at (147.3, 142.1)
- added H5: MountingHole_Pad, MountingHole:MountingHole_2.2mm_M2_Pad_Via, F.Cu at (141.6, 63.6)
- added H6: MountingHole_Pad, MountingHole:MountingHole_2.2mm_M2_Pad_Via, F.Cu at (141.6, 53.3)
- added H7: MountingHole_Pad, MountingHole:MountingHole_2.2mm_M2_Pad_Via, F.Cu at (130.8, 73.4)
- added H8: MountingHole_Pad, MountingHole:MountingHole_2.2mm_M2_Pad_Via, F.Cu at (130.8, 83.6)
- added H9: MountingHole_Pad, MountingHole:MountingHole_2.2mm_M2_Pad_Via, F.Cu at (141.6, 73.4)
- H1, H2, H3, H4: value MountingHole_Pad_MP -> MountingHole_Pad
- U1: footprint PGA-103+:DF782_MNC -> Package_TO_SOT_SMD:SOT-89-3_Handsoldering
- moved J8 146.3 mm to (159.4, 132.1)
- moved J6 146.2 mm to (159.3, 102.6)
- moved J4 146.1 mm to (159.2, 78.4)
- moved J5 124.6 mm to (137.4, 102.6), turned to 180 degrees
- moved J7 123.2 mm to (135.5, 132.1), turned to 180 degrees
- moved C14 120.6 mm to (150.2, 78.5)
- moved C12 113.6 mm to (146.2, 79.2), turned to 90 degrees
- moved J3 111.7 mm to (124.4, 78.5), turned to 180 degrees
- moved C11 108.6 mm to (140.4, 78.5)
- moved L11 106.2 mm to (143.6, 78.5)
- moved L14 102.4 mm to (153.5, 78.5)
- moved C21 101.9 mm to (159.4, 123.8), turned to 90 degrees
- moved C9 101.5 mm to (136.3, 79.3), turned to 90 degrees
- moved L9 99.4 mm to (138.0, 77.4), turned to 90 degrees
- moved L13 97.7 mm to (147.8, 77.4), turned to 90 degrees
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Connections:
- H1 pad 1: (no net) -> GND
- H2 pad 1: (no net) -> GND
- H3 pad 1: (no net) -> GND
- H4 pad 1: (no net) -> GND
Routing:
- net +5V: track 0.00 -> 18.6 mm
- net Net-(C15-Pad2): track 0.00 -> 7.12 mm
- net Net-(J6-In): track 0.00 -> 6.68 mm
- net Net-(C10-Pad2): track 0.00 -> 6.43 mm
- net Net-(J5-In): track 0.00 -> 6.31 mm
- net Net-(U1-RF-OUT/DC-IN): track 0.00 -> 5.79 mm
- net Net-(J3-In): track 0.00 -> 4.87 mm
- net Net-(J7-In): track 0.00 -> 4.57 mm
- net Net-(J8-In): track 0.00 -> 4.57 mm
- net Net-(J4-In): track 0.00 -> 4.32 mm
- net Net-(C12-Pad2): track 0.00 -> 4.31 mm
- net Net-(C11-Pad1): track 0.00 -> 4.30 mm
- net Net-(U1-RF-IN): track 0.00 -> 1.90 mm
- net Net-(C16-Pad1): track 0.00 -> 1.49 mm
- net Net-(C13-Pad1): track 0.00 -> 1.49 mm
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Other:
- board size 35.4 x 14.9 mm -> 40.3 x 94.2 mm
- board text added: "BOT"
- board text added: "TOP"
