File: discrete_filter_board/generic_filt_v1/generic_filt_v1.kicad_sch (KiCad schematic)
At the start: 40 parts, among them J1 Conn_Coaxial, J2 Conn_Coaxial, J3 Conn_Coaxial, J4 Conn_Coaxial, J5 Conn_Coaxial, J6 Conn_Coaxial

Commit message: bpf design
Parts:
- added C18, C19: 0.01 u, Capacitor_SMD:C_0805_2012Metric, symbol Device:C_Small
- added C20: 0.1u, Capacitor_SMD:C_0603_1608Metric, symbol Device:C_Small
- added C21: 10u, Capacitor_SMD:C_1206_3216Metric, symbol Device:C_Small
- added C22: 1 u, Capacitor_SMD:C_0805_2012Metric, symbol Device:C_Small
- added H1, H2, H3, H4: MountingHole_Pad_MP, MountingHole:MountingHole_2.2mm_M2_Pad_Via, symbol Mechanical:MountingHole_Pad_MP
- added J7, J8: Conn_Coaxial, Connector_Coaxial:SMA_Amphenol_132289_EdgeMount, symbol Connector:Conn_Coaxial
- added L18: 10 uH, Inductor_SMD:L_1210_3225Metric, symbol Device:L_Small
- added U1: PGA-103+, PGA-103+:DF782_MNC, symbol PGA-103+:PGA-103+
- C1, C10, C11, C12, C13, C14, C15, C16, C17, C2, C3, C4, C5, C6, C7, C8, C9: footprint (none) -> Capacitor_SMD:C_0603_1608Metric
- J1, J2, J3, J4, J5, J6: footprint (none) -> Connector_Coaxial:SMA_Amphenol_132289_EdgeMount
- L1, L10, L11, L12, L13, L14, L15, L16, L17, L2, L3, L4, L5, L6, L7, L8, L9: footprint (none) -> Inductor_SMD:L_0805_2012Metric
Connections:
- net GND: now also C20.1, C21.1, C22.1, H1.MP, H2.MP, H3.MP, H4.MP, J7.2 (Ext), J8.2 (Ext), U1.2 (GROUND)
- new net: C19.2, J8.1 (In)
- new net: C19.1, L18.2, U1.3 (RF-OUT/DC-IN)
- new net: C18.2, U1.1 (RF-IN)
- new net: C18.1, J7.1 (In)
- new net +5V: C20.2, C21.2, C22.2, L18.1
Other:
- note added: "Order-5 Band Reject filter"
- moved on the sheet: C1, C10, C11, C12, C13, C14, C15, C16, C17, C2, C3, C4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

Commit message: completed pcb routing
Parts:
- removed H1, H2, H3, H4: MountingHole_Pad_MP, MountingHole:MountingHole_2.2mm_M2_Pad_Via, symbol Mechanical:MountingHole_Pad_MP
- added H1, H10, H11, H12, H13, H14, H15, H16, H17, H18, H19, H2, H20, H21, H22, H23, H3, H4, H5, H6, H7, H8, H9: MountingHole_Pad, MountingHole:MountingHole_2.2mm_M2_Pad_Via, symbol Mechanical:MountingHole_Pad
- U1: footprint PGA-103+:DF782_MNC -> Package_TO_SOT_SMD:SOT-89-3_Handsoldering
Connections:
- net GND: now also H1.1, H10.1, H11.1, H12.1, H13.1, H14.1, H15.1, H16.1, H17.1, H18.1, H19.1, H2.1, H20.1, H21.1, H22.1, H23.1, H3.1, H4.1, H5.1, H6.1, H7.1, H8.1, H9.1
